Commit message: Add gripper model and moveit config

File: arctos_description/urdf/arctos.urdf (robot description, URDF)
Before this commit: robot arctos, 8 links, 7 joints
Links:
- added link gripper_body, mass 0.043421; collision mesh filename=package://arctos_description/meshes/gripper_body.STL; visual mesh filename=package://arctos_description/meshes/gripper_body.STL
- added link left_finger, mass 0.011241; collision mesh filename=package://arctos_description/meshes/left_finger.STL; visual mesh filename=package://arctos_description/meshes/left_finger.STL
- added link right_finger, mass 0.011241; collision mesh filename=package://arctos_description/meshes/right_finger.STL; visual mesh filename=package://arctos_description/meshes/right_finger.STL
Joints:
- added joint Gripper_joint: type fixed, parent link_6, child gripper_body, origin xyz=2.2508E-05 0.001025 0.051 rpy=0.0 0.0 0.0, axis 0 0 0, limit lower=0.0 upper=0.0 effort=0.0 velocity=0.0
- added joint Left_finger_joint: type prismatic, parent gripper_body, child left_finger, origin xyz=-0.02655 0 0.0085 rpy=1.5708 0 -3.1416, axis -1.0 0.0 0.0, limit lower=0.002 upper=0.026 effort=100.0 velocity=100.0, mimic joint=Right_finger_joint
- added joint Right_finger_joint: type prismatic, parent gripper_body, child right_finger, origin xyz=0.02575 0 0.0085 rpy=0.0 0.0 0.0, axis -1.0 0.0 0.0, limit lower=0.002 upper=0.026 effort=100.0 velocity=100.0
- joint B_joint: origin xyz=0 0 0.207 rpy=0 0 0 -> xyz=0 0 0.207 rpy=0 0 3.14159265359

File: arctos_description/urdf/arctos.xacro (robot description, xacro)
@@ -3,5 +3,5 @@
   <xacro:include filename="$(find arctos_description)/urdf/common/materials.xacro" />
   <xacro:include filename="$(find arctos_description)/urdf/common/joint_link.xacro" />
-  <!-- <xacro:include filename="$(find arctos_description)/urdf/arctos_gripper.xacro" /> -->
+  <xacro:include filename="$(find arctos_description)/urdf/arctos_gripper.xacro" />
   <link name="world" />
   <joint name="world_joint" type="fixed">
@@ -98,5 +98,5 @@
     name="B_joint" type="revolute"
     parent="link_4" child="link_5"
-    origin_xyz="0 0 0.207" origin_rpy="0 0 0"
+    origin_xyz="0 0 0.207" origin_rpy="0 0 3.14159265359"
     axis_xyz="1 0 0"
     limit_l="-2.0944" limit_u="2.0944" limit_e="1" limit_v="5.236" mimic=""

File: arctos_description/urdf/arctos_gripper.xacro (robot description, xacro)
@@ -5,47 +5,62 @@
   <!-- this definition used the "macro" in urdf/common to quickly define all the attributes-->
   <xacro:arctos_link
-    name="Gripper_1"
-    origin_xyz="-0.000193 0.319847 -0.570316" origin_rpy="0 0 0"
+    name="gripper_body"
+    inertia_origin_xyz="-7.0332E-05 9.1246E-05 -0.0028502" inertia_origin_rpy="0.0 0.0 0.0"
+    mass="0.043421"
+    ixx="7.2269E-06"
+    iyy="3.9281E-05"
+    izz="4.2669E-05"
+    ixy="5.8062E-08"
+    iyz="3.3981E-07"
+    ixz="-5.7636E-08"
+    origin_xyz="0.0 0.0 0.0" origin_rpy="0.0 0.0 0.0"
     material_name="white"
-    inertia_origin_xyz="0.0036112727264542635 -0.014760653808445767 -0.00103677815369696" inertia_origin_rpy="0 0 0"
-    mass="0.5810486809925093"
-    ixx="0.000385" iyy="0.000495" izz="0.000263" ixy="1e-05" iyz="-2e-06" ixz="3e-06"
+  />
+    <xacro:arctos_link
+    name="right_finger"
+    inertia_origin_xyz="0.0093854 2.231E-05 0.024961" inertia_origin_rpy="0.0 0.0 0.0"
+    mass="0.011241"
+    ixx="2.3523E-06"
+    iyy="2.0221E-06"
+    izz="6.0068E-07"
+    ixy="9.9484E-10"
+    iyz="6.0211E-09"
+    ixz="-5.1106E-08"
+    origin_xyz="0.0 0.0 0.0" origin_rpy="0.0 0.0 0.0"
+    material_name="white"
   />
   <xacro:arctos_link
-    name="Left_jaw_1"
-    origin_xyz="-0.007934 0.359845 -0.599867" origin_rpy="0 0 0"
+    name="left_finger"
+    inertia_origin_xyz="0.0093854 0.024961 -2.231E-05" inertia_origin_rpy="0.0 0.0 0.0"
+    mass="0.011241"
+    ixx="2.3523E-06"
+    iyy="6.0068E-07"
+    izz="2.0221E-06"
+    ixy="-5.1106E-08"
+    iyz="-6.0211E-09"
+    ixz="-9.9484E-10"
+    origin_xyz="0.0 0.0 0.0" origin_rpy="0.0 0.0 0.0"
     material_name="white"
-    inertia_origin_xyz="-0.011142702480351952 -0.009692440309284511 -0.009385792627785827" inertia_origin_rpy="0 0 0"
-    mass="0.07369602565859415"
-    ixx="1.1e-05" iyy="6e-06" izz="1.4e-05" ixy="2e-06" iyz="-0.0" ixz="-0.0"
-  />
-  <xacro:arctos_link
-    name="Right_jaw_1"
-    origin_xyz="-0.007934 0.359845 -0.539867" origin_rpy="0 0 0"
-    material_name="white"
-    inertia_origin_xyz="-0.008289104952972526 -0.009768535307719373 0.009395511902715814" inertia_origin_rpy="0 0 0"
-    mass="0.07312902168719511"
-    ixx="1.1e-05" iyy="6e-06" izz="1.4e-05" ixy="-1e-06" iyz="0.0" ixz="-1e-06"
   />
   <!-- Fixed gripper joint, no axis needed -->
   <xacro:arctos_joint
     name="Gripper_joint" type="fixed"
-    parent="Link_6_1" child="Gripper_1"
-    origin_xyz="0.0 -0.006085 0.0" origin_rpy="0 0 0"
+    parent="link_6" child="gripper_body"
+    origin_xyz="2.2508E-05 0.001025 0.051" origin_rpy="0.0 0.0 0.0"
     limit_u="0.0" limit_l="0.0" limit_e="0.0" limit_v="0.0" mimic=""
   />
-  <!-- Left jaw joint, prismatic with axis directly defined -->
+  <!-- Right_finger_joint, prismatic with axis directly defined -->
   <!-- TODO: Movement inverted -->
   <xacro:arctos_joint
-    name="Left_jaw_joint" type="prismatic"
-    parent="Gripper_1" child="Left_jaw_1"
-    origin_xyz="0.007741 -0.039998 0.029551" origin_rpy="0 0 0" axis_xyz="-0.0 0.0 -1.0"
-    limit_u="0.015" limit_l="0.0" limit_e="100.0" limit_v="100.0" mimic=""
+    name="Right_finger_joint" type="prismatic"
+    parent="gripper_body" child="right_finger"
+    origin_xyz="0.02575 0 0.0085" origin_rpy="0.0 0.0 0.0" axis_xyz="-1.0 0.0 0.0"
+    limit_u="0.026" limit_l="0.002" limit_e="100.0" limit_v="100.0" mimic=""
   />
   <xacro:arctos_joint
-    name="Right_jaw_joint" type="prismatic"
-    parent="Gripper_1" child="Right_jaw_1"
-    origin_xyz="0.007741 -0.039998 -0.030449" origin_rpy="0 0 0" axis_xyz="0.0 -0.0 1.0"
-    limit_u="0.015" limit_l="0.0" limit_e="100.0" limit_v="100.0" mimic="Left_jaw_joint"
+    name="Left_finger_joint" type="prismatic"
+    parent="gripper_body" child="left_finger"
+    origin_xyz="-0.02655 0 0.0085" origin_rpy="1.5708 0 -3.1416" axis_xyz="-1.0 0.0 0.0"
+    limit_u="0.026" limit_l="0.002" limit_e="100.0" limit_v="100.0" mimic="Right_finger_joint"
   />
 </robot>

File: arctos_moveit_config/config/arctos.ros2_control.xacro (robot description, xacro)
@@ -2,5 +2,7 @@
 <robot xmlns:xacro="http://www.ros.org/wiki/xacro">
   <xacro:macro name="arctos_ros2_control" params="name initial_positions_file sim:=false">
-    <!--xacro.load_yaml must be used instead of load_yaml, or else we gonna get error: Using load_yaml() directly is deprecated. Use xacro.load_yaml() instead.-->
+    <!--xacro.load_yaml
+    must be used instead of load_yaml, or else we gonna get error: Using load_yaml() directly is
+    deprecated. Use xacro.load_yaml() instead.-->
     <xacro:property name="initial_positions"
       value="${xacro.load_yaml(initial_positions_file)['initial_positions']}" />
@@ -102,4 +104,15 @@
         <state_interface name="velocity" />
       </joint>
+      <joint name="Right_finger_joint">
+        <command_interface name="position">
+          <param name="min">0.002</param>
+          <param name="max">0.026</param>
+        </command_interface>
+        <command_interface name="velocity" />
+        <state_interface name="position">
+          <param name="initial_value">${initial_positions['Right_finger_joint']}</param>
+        </state_interface>
+        <state_interface name="velocity" />
+      </joint>
     </ros2_control>
   </xacro:macro>
