Commit message: action server for Pose movevement + seperate friction/damper for joint

File: arctos_description/urdf/arctos.xacro (robot description, xacro)
@@ -72,5 +72,5 @@
     origin_xyz="0 0 0.183" origin_rpy="0 0 0"
     axis_xyz="0 0 1"
-    limit_l="-2.9671" limit_u="2.9671"  limit_e="1" limit_v="3.0543" mimic=""
+    limit_l="-2.9671" limit_u="2.9671"  limit_e="1" limit_v="3.0543" damping="1.0" friction="0.5" mimic=""
   />
   <xacro:arctos_joint
@@ -79,5 +79,5 @@
     origin_xyz="-0.048 0.075 0.15" origin_rpy="0 0 0"
     axis_xyz="-1 0 0"
-    limit_l="-1.7453" limit_u="2.3562" limit_e="1" limit_v="3.4907" mimic=""
+    limit_l="-1.7453" limit_u="2.3562" limit_e="1" limit_v="3.4907" damping="1.0" friction="0.5" mimic=""
   />
   <xacro:arctos_joint
@@ -86,5 +86,5 @@
     origin_xyz="0 0.029976 0.36377" origin_rpy="0 0 0"
     axis_xyz="-1 0 0"
-    limit_l="-2.0769" limit_u="2.949606436" limit_e="1" limit_v="3.4907" mimic=""
+    limit_l="-2.0769" limit_u="2.949606436" limit_e="1" limit_v="3.4907" damping="0.5" friction="0.3" mimic=""
   />
   <xacro:arctos_joint
@@ -93,5 +93,5 @@
     origin_xyz="0.048 -0.09 0.198" origin_rpy="0 0 0"
     axis_xyz="0 0 1"
-    limit_l="-3.3161" limit_u="3.3161" limit_e="1" limit_v="5.236" mimic=""
+    limit_l="-3.3161" limit_u="3.3161" limit_e="1" limit_v="5.236" damping="0.1" friction="0.1" mimic=""
   />
   <xacro:arctos_joint
@@ -100,5 +100,5 @@
     origin_xyz="0 0 0.207" origin_rpy="0 0 3.14159265359"
     axis_xyz="1 0 0"
-    limit_l="-2.0944" limit_u="2.0944" limit_e="1" limit_v="5.236" mimic=""
+    limit_l="-2.0944" limit_u="2.0944" limit_e="1" limit_v="5.236" damping="0.05" friction="0.05" mimic=""
   />
   <xacro:arctos_joint
@@ -107,5 +107,5 @@
     origin_xyz="0 0 0.052" origin_rpy="0 0 0"
     axis_xyz="0.0 0.0 1.0"
-    limit_l="-6.2832" limit_u="6.2832" limit_e="1" limit_v="8.3776" mimic=""
+    limit_l="-6.2832" limit_u="6.2832" limit_e="1" limit_v="8.3776" damping="0.01" friction="0.01" mimic=""
   />
 </robot>

File: arctos_description/urdf/arctos_gripper.xacro (robot description, xacro)
@@ -56,5 +56,5 @@
     parent="gripper_body" child="right_finger"
     origin_xyz="0.02575 0 0.0085" origin_rpy="0.0 0.0 0.0" axis_xyz="-1.0 0.0 0.0"
-    limit_u="0.054" limit_l="0.002" limit_e="100.0" limit_v="100.0" mimic=""
+    limit_u="0.054" limit_l="0.002" limit_e="100.0" limit_v="100.0" damping="0.01" friction="0.0" mimic=""
   />
   <xacro:arctos_joint
@@ -62,5 +62,5 @@
     parent="gripper_body" child="left_finger"
     origin_xyz="-0.02655 0 0.0085" origin_rpy="1.5708 0 -3.1416" axis_xyz="-1.0 0.0 0.0"
-    limit_u="0.054" limit_l="0.002" limit_e="100.0" limit_v="100.0" mimic="Right_finger_joint"
+    limit_u="0.054" limit_l="0.002" limit_e="100.0" limit_v="100.0" damping="0.01" friction="0.0" mimic="Right_finger_joint"
   />
 </robot>

File: arctos_description/urdf/common/joint_link.xacro (robot description, xacro)
@@ -34,5 +34,5 @@
   <!-- TODO: Add param for mechanicalReduction -->
   <xacro:macro name="arctos_joint"
-    params="name type parent child origin_xyz origin_rpy axis_xyz='0 0 0' limit_u limit_l limit_e limit_v mimic">
+    params="name type parent child origin_xyz origin_rpy axis_xyz='0 0 0' limit_u limit_l limit_e limit_v damping friction mimic">
     <joint name="${name}" type="${type}">
       <parent link="${parent}" />
@@ -42,9 +42,9 @@
       <limit upper="${limit_u}" lower="${limit_l}" effort="${limit_e}" velocity="${limit_v}" />
       <xacro:if value="${mimic != ''}">
-        <mimic joint="${mimic}" />
+        <mimic joint="${mimic}" multiplier="1.0" offset="0.0"/>
       </xacro:if>
-      <dynamics damping="2.0" friction="0.2"/>
+      <dynamics damping="${damping}" friction="${friction}"/>
     </joint>
-    <xacro:if value="${mimic != ''}">
+    <xacro:if value="${mimic == ''}">
       <!-- Add transmission element -->
       <transmission name="transmission_${name}">

Commit message: Update the model with new gripper type

File: arctos_description/urdf/arctos.xacro (robot description, xacro)
@@ -14,5 +14,10 @@
     inertia_origin_xyz="-0.00047006 -0.012257 0.10022" inertia_origin_rpy="0 0 0"
     mass="55.785"
-    ixx="0.39179" ixy="-0.0027323" ixz="-0.00075955" iyy="0.323" iyz="-0.022558" izz="0.34492"
+    ixx="0.39179"
+        ixy="-0.0027323"
+        ixz="-0.00075955"
+        iyy="0.323"
+        iyz="-0.022558"
+        izz="0.34492"
     origin_xyz="0 0 0" origin_rpy="0 0 0"
     material_name="base_blue"
@@ -22,5 +27,10 @@
     inertia_origin_xyz="0.0075871 0.03734 0.10645" inertia_origin_rpy="0 0 0"
     mass="44.267"
-    ixx="0.28548" ixy="-0.012987" ixz="-0.013929" iyy="0.25047" iyz="-0.073189" izz="0.26167"
+    ixx="0.28548"
+        ixy="-0.012987"
+        ixz="-0.013929"
+        iyy="0.25047"
+        iyz="-0.073189"
+        izz="0.26167"
     origin_xyz="0 0 0" origin_rpy="0 0 0"
     material_name="blue"
@@ -28,7 +38,12 @@
   <xacro:arctos_link
     name="link_2"
-    inertia_origin_xyz="-0.068044 0.021826 0.15762" inertia_origin_rpy="0 0 0"
+    inertia_origin_xyz="-0.068043780087778 0.014140910340166 0.158490980475755" inertia_origin_rpy="0 0 0"
     mass="43.339"
-    ixx="0.97722" ixy="0.00042244" ixz="-0.021124" iyy="0.93504" iyz="-0.078229" izz="0.099171"
+    ixx="0.977219187562445"
+        ixy="0.00144844221271251"
+        ixz="-0.021078642737214"
+        iyy="0.940664030252845"
+        iyz="-0.0372886990528127"
+        izz="0.0935514301099311"
     origin_xyz="0 0 0" origin_rpy="0 0 0"
     material_name="gray"
@@ -38,5 +53,10 @@
     inertia_origin_xyz="0.054747 -0.045778 0.060447" inertia_origin_rpy="0 0 0"
     mass="37.594"
-    ixx="0.31727" ixy="-0.0048815" ixz="0.0065087" iyy="0.26582" iyz="0.088578" izz="0.16116"
+    ixx="0.31727"
+        ixy="-0.0048815"
+        ixz="0.0065087"
+        iyy="0.26582"
+        iyz="0.088578"
+        izz="0.16116"
     origin_xyz="0 0 0" origin_rpy="0 0 0"
     material_name="gray"
@@ -46,5 +66,10 @@
     inertia_origin_xyz="0.0051846 -0.00064606 0.10645" inertia_origin_rpy="0 0 0"
     mass="14.917"
-    ixx="0.062769" ixy="3.6977E-05" ixz="-0.001868" iyy="0.069443" iyz="-0.00032273" izz="0.028683"
+    ixx="0.062769"
+        ixy="3.6977E-05"
+        ixz="-0.001868"
+        iyy="0.069443"
+        iyz="-0.00032273"
+        izz="0.028683"
     origin_xyz="0 0 0" origin_rpy="0 0 0"
     material_name="gray"
@@ -54,5 +79,10 @@
     inertia_origin_xyz="-0.00049422 2.4246E-07 0.0067098" inertia_origin_rpy="0 0 0"
     mass="0.34309"
-    ixx="0.00034995" ixy="-1.2487E-09" ixz="-1.1371E-06" iyy="0.00030039" iyz="-1.4302E-09" izz="0.00022745"
+    ixx="0.00034995"
+        ixy="-1.2487E-09"
+        ixz="-1.1371E-06"
+        iyy="0.00030039"
+        iyz="-1.4302E-09"
+        izz="0.00022745"
     origin_xyz="0 0 0" origin_rpy="0 0 0"
     material_name="gray"
@@ -60,7 +90,12 @@
   <xacro:arctos_link
     name="link_6"
-    inertia_origin_xyz="3.1972E-05 -5.2042E-18 0.011587" inertia_origin_rpy="0.0 0.0 0.0"
+    inertia_origin_xyz="3.1956E-05 1.0191E-06 0.011587" inertia_origin_rpy="0.0 0.0 0.0"
     mass="0.068739"
-    ixx="2.0617E-05" ixy="-1.6907E-20" ixz="-2.849E-08" iyy="2.0453E-05" iyz="2.0027E-21" izz="3.4376E-05"
+    ixx="2.0616E-05"
+        ixy="5.2203E-09"
+        ixz="-2.8476E-08"
+        iyy="2.0453E-05"
+        iyz="-9.0808E-10"
+        izz="3.4376E-05"
     origin_xyz="0 0 0" origin_rpy="0 0 0"
     material_name="gray"
@@ -84,5 +119,5 @@
     name="Z_joint" type="revolute"
     parent="link_2" child="link_3"
-    origin_xyz="0 0.029976 0.36377" origin_rpy="0 0 0"
+    origin_xyz="0 0.012264 0.36479" origin_rpy="0 0 0"
     axis_xyz="-1 0 0"
     limit_l="-2.0769" limit_u="2.949606436" limit_e="1" limit_v="3.4907" damping="0.5" friction="0.3" mimic=""
@@ -98,5 +133,5 @@
     name="B_joint" type="revolute"
     parent="link_4" child="link_5"
-    origin_xyz="0 0 0.207" origin_rpy="0 0 3.14159265359"
+    origin_xyz="0 0 0.207" origin_rpy="0 0 3.14159265358979"
     axis_xyz="1 0 0"
     limit_l="-2.0944" limit_u="2.0944" limit_e="1" limit_v="5.236" damping="0.05" friction="0.05" mimic=""

File: arctos_description/urdf/arctos_gripper.xacro (robot description, xacro)
@@ -5,62 +5,103 @@
   <!-- this definition used the "macro" in urdf/common to quickly define all the attributes-->
   <xacro:arctos_link
-    name="gripper_body"
-    inertia_origin_xyz="-0.00019585 -0.016421 0.020172" inertia_origin_rpy="0.0 0.0 0.0"
-    mass="0.33417"
-    ixx="0.00022453"
-    ixy="-3.0847E-05"
-    ixz="-2.1052E-06"
-    iyy="0.0012489"
-    iyz="9.1658E-06"
-    izz="0.001362"
+    name="gripper_body_link"
+    inertia_origin_xyz="0.00020982 0.003292 0.033301" inertia_origin_rpy="0.0 0.0 0.0"
+    mass="0.0054091"
+    ixx="2.85E-06"
+    ixy="1E-08"
+    ixz="-1E-08"
+    iyy="3.53E-06"
+    iyz="-3.5E-07"
+    izz="1.92E-06"
     origin_xyz="0.0 0.0 0.0" origin_rpy="0.0 0.0 0.0"
-    material_name="white"
-  />
-    <xacro:arctos_link
-    name="right_finger"
-    inertia_origin_xyz="0.04544 -0.014371 0.082448" inertia_origin_rpy="0.0 0.0 0.0"
-    mass="0.089929"
-    ixx="7.526E-05"
-    ixy="3.6832E-07"
-    ixz="-1.6407E-06"
-    iyy="6.4721E-05"
-    iyz="1.4045E-07"
-    izz="1.9222E-05"
-    origin_xyz="0.0 0.0 0.0" origin_rpy="0.0 0.0 0.0"
-    material_name="white"
+    material_name="shiny_black"
   />
   <xacro:arctos_link
-    name="left_finger"
-    inertia_origin_xyz="0.045526 0.082448 -0.019029" inertia_origin_rpy="0.0 0.0 0.0"
-    mass="0.089929"
-    ixx="7.526E-05"
-    ixy="-1.6407E-06"
-    ixz="-3.6832E-07"
-    iyy="1.9222E-05"
-    iyz="-1.4045E-07"
-    izz="6.4721E-05"
+    name="gripper_gear_right"
+    inertia_origin_xyz="-0.00035596 -0.0024435 0.018593" inertia_origin_rpy="0.0 0.0 0.0"
+    mass="0.0019306"
+    ixx="7.1E-07"
+    ixy="0.0"
+    ixz="-1E-08"
+    iyy="7.4E-07"
+    iyz="-1E-08"
+    izz="4E-08"
     origin_xyz="0.0 0.0 0.0" origin_rpy="0.0 0.0 0.0"
-    material_name="white"
+    material_name="shiny_black"
+  />
+  <xacro:arctos_link
+    name="gripper_head_right"
+    inertia_origin_xyz="0.0041166 -0.0074512 0.016822" inertia_origin_rpy="0.0 0.0 0.0"
+    mass="0.0063243"
+    ixx="2.31E-06"
+    ixy="0.0"
+    ixz="4.4E-07"
+    iyy="1.61E-06"
+    iyz="0.0"
+    izz="1.26E-06"
+    origin_xyz="0.0 0.0 0.0" origin_rpy="0.0 0.0 0.0"
+    material_name="shiny_black"
+  />
+  <xacro:arctos_link
+    name="gripper_gear_left"
+    inertia_origin_xyz="0.00022186 -0.0024435 0.018595" inertia_origin_rpy="0.0 0.0 0.0"
+    mass="0.0019306"
+    ixx="7.1E-07"
+    ixy="0.0"
+    ixz="1E-08"
+    iyy="7.4E-07"
+    iyz="-1E-08"
+    izz="4E-08"
+    origin_xyz="0.0 0.0 0.0" origin_rpy="0.0 0.0 0.0"
+    material_name="shiny_black"
+  />
+  <xacro:arctos_link
+    name="gripper_head_left"
+    inertia_origin_xyz="-0.0041166 -0.0074512 0.016822" inertia_origin_rpy="0.0 0.0 0.0"
+    mass="0.0063243"
+    ixx="2.31E-06"
+    ixy="0.0"
+    ixz="-4.4E-07"
+    iyy="1.61E-06"
+    iyz="0.0"
+    izz="1.26E-06"
+    origin_xyz="0.0 0.0 0.0" origin_rpy="0.0 0.0 0.0"
+    material_name="shiny_black"
   />
   <!-- Fixed gripper joint, no axis needed -->
   <xacro:arctos_joint
-    name="Gripper_joint" type="fixed"
-    parent="link_6" child="gripper_body"
-    origin_xyz="2.2508E-05 0.001025 0.051" origin_rpy="0.0 0.0 0.0"
+    name="gripper_body_joint" type="fixed"
+    parent="link_6" child="gripper_body_link"
+    origin_xyz="0 0 0.0219999999999994" origin_rpy="0.0 0.0 3.14159265358979"
     limit_u="0.0" limit_l="0.0" limit_e="0.0" limit_v="0.0" damping="0.0" friction="0.0" mimic=""
   />
-  <!-- Right_finger_joint, prismatic with axis directly defined -->
-  <!-- TODO: Movement inverted -->
+  <!-- gripper_gear_right_joint, revolute with axis directly defined -->
   <xacro:arctos_joint
-    name="Right_finger_joint" type="prismatic"
-    parent="gripper_body" child="right_finger"
-    origin_xyz="0.02575 0 0.0085" origin_rpy="0.0 0.0 0.0" axis_xyz="-1.0 0.0 0.0"
-    limit_u="0.054" limit_l="0.002" limit_e="100.0" limit_v="100.0" damping="0.02" friction="0.0" mimic=""
+    name="gripper_gear_right_joint" type="revolute"
+    parent="gripper_body_link" child="gripper_gear_right"
+    origin_xyz="-0.0105000000000263 0.0175575664610773 0.0484957779974575" origin_rpy="0.0 0.0 0.0"
+    axis_xyz="0.0 -1.0 0.0"
+    limit_u="1.4835" limit_l="0.0175" limit_e="100.0" limit_v="100.0" damping="0.02" friction="0.0"
+    mimic=""
   />
   <xacro:arctos_joint
-    name="Left_finger_joint" type="prismatic"
-    parent="gripper_body" child="left_finger"
-    origin_xyz="-0.02655 0 0.0085" origin_rpy="1.5708 0 -3.1416" axis_xyz="-1.0 0.0 0.0"
-    limit_u="0.054" limit_l="0.002" limit_e="100.0" limit_v="100.0" damping="0.02" friction="0.0" mimic="Right_finger_joint"
+    name="gripper_head_right_joint" type="fixed"
+    parent="gripper_gear_right" child="gripper_head_right"
+    origin_xyz="-0.000818014467841976 0 0.043192254540952" origin_rpy="0.0 0.0 0.0"
+    limit_u="0.0" limit_l="0.0" limit_e="0.0" limit_v="0.0" damping="0.0" friction="0.0" mimic=""
+  />
+  <xacro:arctos_joint
+    name="gripper_gear_left_joint" type="revolute"
+    parent="gripper_body_link" child="gripper_gear_left"
+    origin_xyz="0.0105 0.017558 0.048496" origin_rpy="0.0 0.0 0.0"
+    axis_xyz="0.0 1.0 0.0"
+    limit_u="1.4835" limit_l="0.0175" limit_e="100.0" limit_v="100.0" damping="0.02" friction="0.0"
+    mimic="gripper_gear_right_joint"
+  />
+  <xacro:arctos_joint
+    name="gripper_head_left_joint" type="fixed"
+    parent="gripper_gear_left" child="gripper_head_left"
+    origin_xyz="0.000524248952185996 0 0.0431968188995016" origin_rpy="0.0 0.0 0.0"
+    limit_u="0.0" limit_l="0.0" limit_e="0.0" limit_v="0.0" damping="0.0" friction="0.0" mimic=""
   />
 </robot>

File: arctos_description/urdf/common/materials.xacro (robot description, xacro)
@@ -6,4 +6,7 @@
   <material name="black">
     <color rgba="0.0 0.0 0.0 1.0" />
+  </material>
+  <material name="shiny_black">
+    <color rgba="0.79216 0.81961 0.93333 1.0" />
   </material>
   <material name="base_blue">

File: arctos_moveit_config/config/arctos.ros2_control.xacro (robot description, xacro)
@@ -74,19 +74,19 @@
         </state_interface>
       </joint>
-      <joint name="Right_finger_joint">
+      <joint name="gripper_gear_right_joint">
         <command_interface name="position">
-          <param name="min">0.002</param>
-          <param name="max">0.054</param>
+          <param name="min">0.0175</param>
+          <param name="max">1.4835</param>
         </command_interface>
         <state_interface name="position">
-          <param name="initial_value">${initial_positions['Right_finger_joint']}</param>
+          <param name="initial_value">${initial_positions['gripper_gear_right_joint']}</param>
         </state_interface>
         <state_interface name="velocity" />
       </joint>
-      <!-- <joint name="Left_finger_joint">
-        <param name="mimic">Right_finger_joint</param>
+      <!-- <joint name="gripper_gear_left_joint">
+        <param name="mimic">gripper_gear_right_joint</param>
         <param name="multiplier">1</param>
         <state_interface name="position">
-          <param name="initial_value">${initial_positions['Right_finger_joint']}</param>
+          <param name="initial_value">${initial_positions['gripper_gear_right_joint']}</param>
         </state_interface>
         <state_interface name="velocity" />

Commit message: Limit joint 5 to avoid break the end-effector

File: arctos_description/urdf/arctos.xacro (robot description, xacro)
@@ -6,6 +6,6 @@
   <link name="world" />
   <joint name="world_joint" type="fixed">
-      <parent link="world"/>
-      <child link="base_link"/>
+    <parent link="world" />
+    <child link="base_link" />
   </joint>
   <!-- Define all links -->
@@ -15,9 +15,9 @@
     mass="55.785"
     ixx="0.39179"
-        ixy="-0.0027323"
-        ixz="-0.00075955"
-        iyy="0.323"
-        iyz="-0.022558"
-        izz="0.34492"
+    ixy="-0.0027323"
+    ixz="-0.00075955"
+    iyy="0.323"
+    iyz="-0.022558"
+    izz="0.34492"
     origin_xyz="0 0 0" origin_rpy="0 0 0"
     material_name="base_blue"
@@ -28,9 +28,9 @@
     mass="44.267"
     ixx="0.28548"
-        ixy="-0.012987"
-        ixz="-0.013929"
-        iyy="0.25047"
-        iyz="-0.073189"
-        izz="0.26167"
+    ixy="-0.012987"
+    ixz="-0.013929"
+    iyy="0.25047"
+    iyz="-0.073189"
+    izz="0.26167"
     origin_xyz="0 0 0" origin_rpy="0 0 0"
     material_name="blue"
@@ -38,12 +38,13 @@
   <xacro:arctos_link
     name="link_2"
-    inertia_origin_xyz="-0.068043780087778 0.014140910340166 0.158490980475755" inertia_origin_rpy="0 0 0"
+    inertia_origin_xyz="-0.068043780087778 0.014140910340166 0.158490980475755"
+    inertia_origin_rpy="0 0 0"
     mass="43.339"
     ixx="0.977219187562445"
-        ixy="0.00144844221271251"
-        ixz="-0.021078642737214"
-        iyy="0.940664030252845"
-        iyz="-0.0372886990528127"
-        izz="0.0935514301099311"
+    ixy="0.00144844221271251"
+    ixz="-0.021078642737214"
+    iyy="0.940664030252845"
+    iyz="-0.0372886990528127"
+    izz="0.0935514301099311"
     origin_xyz="0 0 0" origin_rpy="0 0 0"
     material_name="gray"
@@ -54,9 +55,9 @@
     mass="37.594"
     ixx="0.31727"
-        ixy="-0.0048815"
-        ixz="0.0065087"
-        iyy="0.26582"
-        iyz="0.088578"
-        izz="0.16116"
+    ixy="-0.0048815"
+    ixz="0.0065087"
+    iyy="0.26582"
+    iyz="0.088578"
+    izz="0.16116"
     origin_xyz="0 0 0" origin_rpy="0 0 0"
     material_name="gray"
@@ -67,9 +68,9 @@
     mass="14.917"
     ixx="0.062769"
-        ixy="3.6977E-05"
-        ixz="-0.001868"
-        iyy="0.069443"
-        iyz="-0.00032273"
-        izz="0.028683"
+    ixy="3.6977E-05"
+    ixz="-0.001868"
+    iyy="0.069443"
+    iyz="-0.00032273"
+    izz="0.028683"
     origin_xyz="0 0 0" origin_rpy="0 0 0"
     material_name="gray"
@@ -80,9 +81,9 @@
     mass="0.34309"
     ixx="0.00034995"
-        ixy="-1.2487E-09"
-        ixz="-1.1371E-06"
-        iyy="0.00030039"
-        iyz="-1.4302E-09"
-        izz="0.00022745"
+    ixy="-1.2487E-09"
+    ixz="-1.1371E-06"
+    iyy="0.00030039"
+    iyz="-1.4302E-09"
+    izz="0.00022745"
     origin_xyz="0 0 0" origin_rpy="0 0 0"
     material_name="gray"
@@ -93,13 +94,14 @@
     mass="0.068739"
     ixx="2.0616E-05"
-        ixy="5.2203E-09"
-        ixz="-2.8476E-08"
-        iyy="2.0453E-05"
-        iyz="-9.0808E-10"
-        izz="3.4376E-05"
+    ixy="5.2203E-09"
+    ixz="-2.8476E-08"
+    iyy="2.0453E-05"
+    iyz="-9.0808E-10"
+    izz="3.4376E-05"
     origin_xyz="0 0 0" origin_rpy="0 0 0"
     material_name="gray"
   />
-  <!--Change limit of joints here-->
+  <!--Change
+  limit of joints here-->
   <xacro:arctos_joint
     name="X_joint" type="revolute"
@@ -107,5 +109,6 @@
     origin_xyz="0 0 0.183" origin_rpy="0 0 0"
     axis_xyz="0 0 1"
-    limit_l="-2.9671" limit_u="2.9671"  limit_e="1" limit_v="3.0543" damping="1.0" friction="0.5" mimic=""
+    limit_l="-2.9671" limit_u="2.9671" limit_e="1" limit_v="3.0543" damping="1.0" friction="0.5"
+    mimic=""
   />
   <xacro:arctos_joint
@@ -114,5 +117,6 @@
     origin_xyz="-0.048 0.075 0.15" origin_rpy="0 0 0"
     axis_xyz="-1 0 0"
-    limit_l="-1.7453" limit_u="2.3562" limit_e="1" limit_v="3.4907" damping="1.0" friction="0.5" mimic=""
+    limit_l="-1.7453" limit_u="2.3562" limit_e="1" limit_v="3.4907" damping="1.0" friction="0.5"
+    mimic=""
   />
   <xacro:arctos_joint
@@ -121,5 +125,6 @@
     origin_xyz="0 0.012264 0.36479" origin_rpy="0 0 0"
     axis_xyz="-1 0 0"
-    limit_l="-2.0769" limit_u="2.949606436" limit_e="1" limit_v="3.4907" damping="0.5" friction="0.3" mimic=""
+    limit_l="-2.0769" limit_u="2.949606436" limit_e="1" limit_v="3.4907" damping="0.5"
+    friction="0.3" mimic=""
   />
   <xacro:arctos_joint
@@ -128,5 +133,6 @@
     origin_xyz="0.048 -0.09 0.198" origin_rpy="0 0 0"
     axis_xyz="0 0 1"
-    limit_l="-3.3161" limit_u="3.3161" limit_e="1" limit_v="5.236" damping="0.1" friction="0.1" mimic=""
+    limit_l="-3.3161" limit_u="3.3161" limit_e="1" limit_v="5.236" damping="0.1" friction="0.1"
+    mimic=""
   />
   <xacro:arctos_joint
@@ -135,5 +141,6 @@
     origin_xyz="0 0 0.207" origin_rpy="0 0 3.14159265358979"
     axis_xyz="1 0 0"
-    limit_l="-2.0944" limit_u="2.0944" limit_e="1" limit_v="5.236" damping="0.05" friction="0.05" mimic=""
+    limit_l="-1.570796" limit_u="1.570796" limit_e="1" limit_v="5.236" damping="0.05" friction="0.05"
+    mimic=""
   />
   <xacro:arctos_joint
@@ -142,5 +149,6 @@
     origin_xyz="0 0 0.052" origin_rpy="0 0 0"
     axis_xyz="0.0 0.0 1.0"
-    limit_l="-6.2832" limit_u="6.2832" limit_e="1" limit_v="8.3776" damping="0.01" friction="0.01" mimic=""
+    limit_l="-6.2832" limit_u="6.2832" limit_e="1" limit_v="8.3776" damping="0.01" friction="0.01"
+    mimic=""
   />
 </robot>
