Commit message: add Gazebo to project and link between gazebo with ros2.

File: arctos_description/urdf/common/joint_link.xacro (robot description, xacro)
@@ -8,5 +8,5 @@
         <origin xyz="${origin_xyz}" rpy="${origin_rpy}" />
         <geometry>
-          <mesh filename="package://arctos_description/meshes/${name}.STL"/>
+          <mesh filename="package://arctos_description/meshes/${name}.STL" />
         </geometry>
         <material name="${material_name}" />
@@ -15,5 +15,5 @@
         <origin xyz="${origin_xyz}" rpy="${origin_rpy}" />
         <geometry>
-          <mesh filename="package://arctos_description/meshes/${name}.STL"/>
+          <mesh filename="package://arctos_description/meshes/${name}.STL" />
         </geometry>
       </collision>
@@ -24,4 +24,10 @@
       </inertial>
     </link>
+    <!-- However, the correct and explicit way when gazebo lives outside the link -->
+    <gazebo reference="${name}">
+      <!-- https://sdformat.org/spec/1.12/link/#link_kinematic -->
+      <kinematic>true</kinematic>
+      <gravity>false</gravity>
+    </gazebo>
   </xacro:macro>
   <!-- Define arctos_joint macro with a default value for axis_xyz -->
@@ -36,6 +42,7 @@
       <limit upper="${limit_u}" lower="${limit_l}" effort="${limit_e}" velocity="${limit_v}" />
       <xacro:if value="${mimic != ''}">
-          <mimic joint="${mimic}" />
+        <mimic joint="${mimic}" />
       </xacro:if>
+      <dynamics damping="2.0" friction="0.2"/>
     </joint>
     <!-- Add transmission element -->
@@ -53,8 +60,8 @@
     <joint name="${name}">
       <command_interface name="position">
-            <param name="min">${limit_l}</param>
-            <param name="max">${limit_u}</param>
+        <param name="min">${limit_l}</param>
+        <param name="max">${limit_u}</param>
       </command_interface>
-      <state_interface name="position"/>
+      <state_interface name="position" />
     </joint>
   </xacro:macro>

File: arctos_moveit_config/config/arctos.ros2_control.xacro (robot description, xacro)
@@ -9,7 +9,7 @@
     <ros2_control name="${name}" type="system">
       <hardware>
-        <!-- By default, set up controllers for simulation. This won't work on real hardware -->
+        <!-- By default, set up controllers for gazebo. This won't work on real hardware -->
         <xacro:if value="${sim}">
-          <plugin>mock_components/GenericSystem</plugin>
+          <plugin>gz_ros2_control/GazeboSimSystem</plugin>
         </xacro:if>
         <xacro:unless value="${sim}">
@@ -84,5 +84,22 @@
         <state_interface name="velocity" />
       </joint>
+      <joint name="Left_finger_joint_mimic">
+        <param name="mimic">Right_finger_joint</param>
+        <param name="multiplier">1</param>
+        <command_interface name="position" />
+        <state_interface name="position">
+          <param name="initial_value">${initial_positions['Right_finger_joint']}</param>
+        </state_interface>
+        <state_interface name="velocity" />
+      </joint>
     </ros2_control>
+    <gazebo>
+      <plugin filename="gz_ros2_control-system" name="gz_ros2_control::GazeboSimROS2ControlPlugin">
+        <robot_param>robot_description</robot_param>
+        <robot_param_node>robot_state_publisher</robot_param_node>
+        <parameters>$(find arctos_moveit_config)/config/ros2_controllers.yaml</parameters>
+        <controller_manager_name>controller_manager</controller_manager_name>
+      </plugin>
+    </gazebo>
   </xacro:macro>
 </robot>

Commit message: working right gripper

File: arctos_description/urdf/common/joint_link.xacro (robot description, xacro)
@@ -46,14 +46,16 @@
       <dynamics damping="2.0" friction="0.2"/>
     </joint>
-    <!-- Add transmission element -->
-    <transmission name="transmission_${name}">
-      <type>transmission_interface/SimpleTransmission</type>
-      <joint name="${name}">
-        <hardwareInterface>hardware_interface/PositionJointInterface</hardwareInterface>
-      </joint>
-      <actuator name="${name}_motor">
-        <mechanicalReduction>1.0</mechanicalReduction>
-      </actuator>
-    </transmission>
+    <xacro:if value="${mimic != ''}">
+      <!-- Add transmission element -->
+      <transmission name="transmission_${name}">
+        <type>transmission_interface/SimpleTransmission</type>
+        <joint name="${name}">
+          <hardwareInterface>hardware_interface/PositionJointInterface</hardwareInterface>
+        </joint>
+        <actuator name="${name}_motor">
+          <mechanicalReduction>1.0</mechanicalReduction>
+        </actuator>
+      </transmission>
+    </xacro:if>
   </xacro:macro>
   <xacro:macro name="arctos_control" params="name limit_u limit_l">

File: arctos_moveit_config/config/arctos.ros2_control.xacro (robot description, xacro)
@@ -84,8 +84,7 @@
         <state_interface name="velocity" />
       </joint>
-      <joint name="Left_finger_joint_mimic">
+      <joint name="Left_finger_joint">
         <param name="mimic">Right_finger_joint</param>
         <param name="multiplier">1</param>
-        <command_interface name="position" />
         <state_interface name="position">
           <param name="initial_value">${initial_positions['Right_finger_joint']}</param>
