Commit message: update for compatibility with real hardware. gazebo can't move left_finger_joint as a result

File: arctos_moveit_config/config/arctos.ros2_control.xacro (robot description, xacro)
@@ -84,5 +84,5 @@
         <state_interface name="velocity" />
       </joint>
-      <joint name="Left_finger_joint">
+      <!-- <joint name="Left_finger_joint">
         <param name="mimic">Right_finger_joint</param>
         <param name="multiplier">1</param>
@@ -91,5 +91,5 @@
         </state_interface>
         <state_interface name="velocity" />
-      </joint>
+      </joint> -->
     </ros2_control>
     <gazebo>

Commit message: Add DensoHandInterface and ServoDriver for Gripper control
- Implemented ServoDriver class to manage servo motors, including methods for adding, removing, and controlling servos.
- Added functionality to process UART messages and update servo states based on encoder feedback.
- Introduced methods for setting servo limits, retrieving positions, and handling motor commands.
- Created configuration file for Denso hand integration with ROS 2 control, specifying hardware parameters and joint interfaces.

File: arctos_moveit_config/config/arctos.ros2_control.xacro (robot description, xacro)
@@ -74,22 +74,4 @@
         </state_interface>
       </joint>
-      <joint name="gripper_gear_right_joint">
-        <command_interface name="position">
-          <param name="min">0.02</param>
-          <param name="max">1.4835</param>
-        </command_interface>
-        <state_interface name="position">
-          <param name="initial_value">${initial_positions['gripper_gear_right_joint']}</param>
-        </state_interface>
-        <state_interface name="velocity" />
-      </joint>
-      <!-- <joint name="gripper_gear_left_joint">
-        <param name="mimic">gripper_gear_right_joint</param>
-        <param name="multiplier">1</param>
-        <state_interface name="position">
-          <param name="initial_value">${initial_positions['gripper_gear_right_joint']}</param>
-        </state_interface>
-        <state_interface name="velocity" />
-      </joint> -->
     </ros2_control>
     <gazebo>

File: arctos_moveit_config/config/arctos.urdf.xacro (robot description, xacro)
@@ -6,4 +6,6 @@
     <!-- Import control_xacro -->
     <xacro:include filename="arctos.ros2_control.xacro" />
+    <xacro:include filename="denso_hand.ros2_control.xacro" />
     <xacro:arctos_ros2_control name="RealSystem" initial_positions_file="$(arg initial_positions_file)" sim="false"/>
+    <xacro:denso_hand_ros2_control name="HandRealSystem" initial_positions_file="$(arg initial_positions_file)" sim="false"/>
 </robot>

File: arctos_moveit_config/config/gz_arctos.urdf.xacro (robot description, xacro)
@@ -6,4 +6,6 @@
     <!-- Import control_xacro -->
     <xacro:include filename="arctos.ros2_control.xacro" />
+    <xacro:include filename="denso_hand.ros2_control.xacro" />
     <xacro:arctos_ros2_control name="GazeboSimSystem" initial_positions_file="$(arg initial_positions_file)" sim="true"/>
+    <xacro:denso_hand_ros2_control name="HandGazeboSimSystem" initial_positions_file="$(arg initial_positions_file)" sim="true"/>
 </robot>
